Commit message: update nav

File: manipulator_description/urdf/accessories/hokuyo_ust-10lx_mount.urdf.xacro (robot description, xacro)
@@ -11,7 +11,5 @@
         <mass value="0.130" />
         <origin xyz="0 0 0" />
-        <inertia ixx="${0.0833333 * 0.130 * (0.05*0.05 + 0.07*0.07)}" ixy="0.0" ixz="0.0"
-          iyy="${0.0833333 * 0.130 * (0.05*0.05 + 0.07*0.07)}" iyz="0.0"
-          izz="${0.0833333 * 0.130 * (0.05*0.05 + 0.05*0.05)}" />
+        <inertia ixx="${0.0833333 * 0.130 * (0.05*0.05 + 0.07*0.07)}" ixy="0.0" ixz="0.0" iyy="${0.0833333 * 0.130 * (0.05*0.05 + 0.07*0.07)}" iyz="0.0" izz="${0.0833333 * 0.130 * (0.05*0.05 + 0.05*0.05)}" />
       </inertial>
       <visual>
@@ -19,5 +17,5 @@
         <geometry>
           <!-- Origin of this mesh is the focal point of the LIDAR. -->
-          <mesh filename="package://ridgeback_description/meshes/ust-10lx.stl" />
+          <mesh filename="package://manipulator_description/meshes/ust-10lx.stl" />
         </geometry>
         <material name="dark_grey" />

File: manipulator_description/urdf/accessories/microstrain_imu.urdf.xacro (robot description, xacro)
@@ -2,36 +2,36 @@
 <robot xmlns:xacro="http://ros.org/wiki/xacro">
   <xacro:macro name="microstrain_imu" params="prefix mount_link *joint_pose">
-  <link name="${prefix}_imu_link" >
-    <visual>
-      <origin xyz="0 0 0" rpy="0 0 0" />
-      <geometry>
-        <!-- Origin of this mesh is the focal point of the LIDAR. -->
-        <mesh filename="package://ridgeback_description/meshes/3dm-gxX.stl" scale="0.001 0.001 0.001" />
-      </geometry>
-      <material name="dark_grey" />
-    </visual>
-  </link>
-  <joint name="${prefix}_imu_joint" type="fixed">
-    <xacro:insert_block name="joint_pose" />
-    <parent link="${mount_link}" />
-    <child link="${prefix}_imu_link" />
-  </joint>
-  <gazebo>
-    <plugin name="${prefix}_imu_controller" filename="libhector_gazebo_ros_imu.so">
-      <robotNamespace>/</robotNamespace>
-      <updateRate>50.0</updateRate>
-      <bodyName>${prefix}_imu_link</bodyName>
-      <topicName>${prefix}_imu/data</topicName>
-      <accelDrift>0.005 0.005 0.005</accelDrift>
-      <accelGaussianNoise>0.005 0.005 0.005</accelGaussianNoise>
-      <rateDrift>0.005 0.005 0.005 </rateDrift>
-      <rateGaussianNoise>0.005 0.005 0.005 </rateGaussianNoise>
-      <headingDrift>0.005</headingDrift>
-      <headingGaussianNoise>0.005</headingGaussianNoise>
-    </plugin>
-  </gazebo>
-  <gazebo reference="${prefix}_imu_link">
-    <material>Gazebo/DarkGrey</material>
-  </gazebo>
+    <link name="${prefix}_imu_link">
+      <visual>
+        <origin xyz="0 0 0" rpy="0 0 0" />
+        <geometry>
+          <!-- Origin of this mesh is the focal point of the LIDAR. -->
+          <mesh filename="package://manipulator_description/meshes/3dm-gxX.stl" scale="0.001 0.001 0.001" />
+        </geometry>
+        <material name="dark_grey" />
+      </visual>
+    </link>
+    <joint name="${prefix}_imu_joint" type="fixed">
+      <xacro:insert_block name="joint_pose" />
+      <parent link="${mount_link}" />
+      <child link="${prefix}_imu_link" />
+    </joint>
+    <gazebo>
+      <plugin name="${prefix}_imu_controller" filename="libhector_gazebo_ros_imu.so">
+        <robotNamespace>/</robotNamespace>
+        <updateRate>50.0</updateRate>
+        <bodyName>${prefix}_imu_link</bodyName>
+        <topicName>${prefix}_imu/data</topicName>
+        <accelDrift>0.005 0.005 0.005</accelDrift>
+        <accelGaussianNoise>0.005 0.005 0.005</accelGaussianNoise>
+        <rateDrift>0.005 0.005 0.005 </rateDrift>
+        <rateGaussianNoise>0.005 0.005 0.005 </rateGaussianNoise>
+        <headingDrift>0.005</headingDrift>
+        <headingGaussianNoise>0.005</headingGaussianNoise>
+      </plugin>
+    </gazebo>
+    <gazebo reference="${prefix}_imu_link">
+      <material>Gazebo/DarkGrey</material>
+    </gazebo>
   </xacro:macro>
 </robot>

File: manipulator_description/urdf/velodyne.urdf.xacro (robot description, xacro)
@@ -37,5 +37,5 @@
         <plugin name="gazebo_ros_laser_controller" filename="libgazebo_ros_velodyne_laser.so">
           <topicName>${topic}</topicName>
-      	  <frameName>${name}</frameName>
+          <frameName>${name}</frameName>
           <min_range>0.9</min_range>
           <max_range>130.0</max_range>
@@ -49,5 +49,5 @@
     <visual>
       <geometry>
-        <mesh filename="package://nuridgeback_description/meshes/vlp16_assy.stl"/>
+        <mesh filename="package://manipulator_description/meshes/vlp16_assy.stl"/>
       </geometry>
       <material name="light_grey">
@@ -57,12 +57,12 @@
     <collision>
       <geometry>
-        <mesh filename="package://nuridgeback_description/meshes/vlp16_assy.stl"/>
+        <mesh filename="package://manipulator_description/meshes/vlp16_assy.stl"/>
       </geometry>
     </collision>
   </link>
   <joint name="base_to_lidar_mesh" type="fixed">
-  <parent link="mid_mount" />
-  <child link="velodyne_mesh" />
-  <origin xyz="0.365 0 0" rpy="0 0 0" />
+    <parent link="mid_mount" />
+    <child link="velodyne_mesh" />
+    <origin xyz="0.365 0 0" rpy="0 0 0" />
   </joint>
   <!-- Create a link between the VLP16 mesh and sensor origin -->
