Commit message: update gui

File: manipulator_description/urdf/sawback.urdf.xacro (robot description, xacro)
@@ -6,4 +6,5 @@
   <xacro:arg name="pedestal" default="false"/>
   <xacro:arg name="static" default="false"/>
+  <xacro:arg name="px100" default="false"/>
   <!-- Ridgeback -->
   <xacro:include filename="$(find manipulator_description)/urdf/nuridgeback.urdf.xacro"/>
@@ -21,3 +22,11 @@
     <child link="base"/>
   </joint>
+  <xacro:if value="$(arg px100)">
+    <xacro:include filename="$(find interbotix_xsarm_descriptions)/urdf/px100.urdf.xacro"/>
+    <joint name="joint_base_to_px100" type="fixed">
+      <parent link="mid_mount"/>
+      <child link="px100/base_link"/>
+      <origin xyz="0.140 -0.3365 0.008" rpy="0.0 0.0 0.0"/>
+    </joint>
+  </xacro:if>
 </robot>
